File: hw/smart-fermentation-glass/smart-fermentation-glass.kicad_sch (KiCad schematic)
At the start: 62 parts, among them IC1 BME688, IC2 VL53L4CDV0DH_1, IC3 MAX17048G+T10, J1 Conn_01x24, J2 Conn_01x02, J603 USB4105-GF-A, Q2 Si1308EDL, SW201 SW_Push, SW202 SW_Push, U2 BQ24074RGT, U3 TPS63031DSK, U4 ESP32-C3-WROOM-02, U602 USBLC6-2SC6

Commit message: completed schematics and pcb
Parts:
- removed L3: VLS5045EX-470M, VLS5045EX330M, symbol custom:VLS5045EX-470M
- added H1, H2: MountingHole_Pad, MountingHole:MountingHole_3.2mm_M3_ISO14580_Pad_TopBottom, symbol Mechanical:MountingHole_Pad
- added L2: SRN4018-470M, SRN4018470M, symbol custom:SRN4018-470M
- C201, C203: footprint Capacitor_SMD:C_0402_1005Metric -> Capacitor_SMD:C_0603_1608Metric
- IC1: footprint BME688 -> custom:BME688
- IC2: footprint VL53L4CDV0DH1 -> custom:VL53L4CDV0DH1
- IC3: footprint SON50P200X200X80-9N-D -> custom:SON50P200X200X80-9N-D
- L1: footprint LQH32CH100K53L -> custom:LQH32CH100K53L
- R202, R203, R204, R205, R206, R207, R208, R601, R602: footprint Resistor_SMD:R_0402_1005Metric -> Resistor_SMD:R_0603_1608Metric
Connections:
- net +3.3V is gone; now on net +3V3: C11.1, C12.1, C14.2, C22.1, C8.1, IC1.2 (CSB), IC1.6 (VDDIO), IC1.8 (VDD), IC3.3 (VDD), J1.15 (Pin_15), J1.16 (Pin_16), R202.2, R203.1, R204.1, R205.2, R206.2, R207.2, R208.2
- net +3V3: now also L2.1
- net BUSY: now also U4.15 (GPIO3/ADC1_CH3); no longer U4.4 (GPIO5/ADC2_CH0)
- net CS: now also U4.5 (GPIO6); no longer U4.16 (GPIO2/ADC1_CH2)
- net D/C: now also U4.6 (GPIO7); no longer U4.15 (GPIO3/ADC1_CH3)
- net GND: now also H1.1, H2.1
- net RST: now also U4.16 (GPIO2/ADC1_CH2); no longer U4.3 (GPIO4/ADC1_CH4)
- net SCLK: now also U4.4 (GPIO5/ADC2_CH0); no longer U4.5 (GPIO6)
- net SDI: now also U4.3 (GPIO4/ADC1_CH4); no longer U4.6 (GPIO7)
- net at C21.2, D4.2 (A), Q2.3 (D): now also L2.2
- no-connect marks 9 -> 10
